File: prue.kicad_sch (KiCad schematic)
At the start: 1 part, among them U1 74AHC240

Commit message: prueba1
Parts:
- added U2: 4001, symbol 4xxx:4001
Changed lines of the file:
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@@
+		)
+	)
+	(symbol
+		(lib_id "4xxx:4001")
+		(at 93.98 140.97 0)
+		(unit 2)
+		(exclude_from_sim no)
+		(in_bom yes)
+		(on_board yes)
+		(dnp no)
+		(fields_autoplaced yes)
+		(property "Reference" "U2"
+			(at 93.98 132.08 0)
+			(effects
+				(font
+					(size 1.27 1.27)
+				)
+			)
+		)
+		(property "Value" "4001"
+			(at 93.98 134.62 0)
+			(effects
+				(font
+					(size 1.27 1.27)
+				)
+			)
+		)
+		(property "Footprint" ""
+			(at 93.98 140.97 0)
+			(effects
+				(font
+					(size 1.27 1.27)
+				)
+				(hide yes)
+			)
+		)
+		(property "Datasheet" "http://www.intersil.com/content/dam/Intersil/documents/cd40/cd4000bms-01bms-02bms-25bms.pdf"
+			(at 93.98 140.97 0)
+			(effects
+				(font
+					(size 1.27 1.27)
+				)
+				(hide yes)
+			)
+		)
+		(property "Description" "Quad Nor 2 inputs"
+			(at 93.98 140.97 0)
+			(effects
+				(font
+					(size 1.27 1.27)
+				)
+				(hide yes)
+			)
+		)
+		(pin "3"
+		)
+		(pin "6"
+		)
+		(pin "4"
+		)
+		(pin "9"
+		)
+		(pin "1"
+		)
+		(pin "12"
+		)
+		(pin "5"
+		)
+		(pin "13"
+		)
+		(pin "2"
+		)
+		(pin "11"
+		)
+		(pin "10"
+		)
+		(pin "8"
+		)
+		(pin "7"
+		)
+		(pin "14"
+		)
+		(instances
+			(project ""
+				(path "/d602fbc7-2a38-4026-b8f4-783c9aa802a9"
+					(reference "U2")
+					(unit 2)
+				)
+			)
+		)
+	)
+	(symbol
+		(lib_id "4xxx:4001")
+		(at 63.5 132.08 0)
+		(unit 1)
+		(exclude_from_sim no)
+		(in_bom yes)
+		(on_board yes)
+		(dnp no)
+		(fields_autoplaced yes)
+		(property "Reference" "U2"
+			(at 63.5 123.19 0)
+			(effects
+				(font
+					(size 1.27 1.27)
+				)
+			)
+		)
+		(property "Value" "4001"
+			(at 63.5 125.73 0)
+			(effects
+				(font
+					(size 1.27 1.27)
+				)
+			)
+		)
+		(property "Footprint" ""
+			(at 63.5 132.08 0)
+			(effects
+				(font
+					(size 1.27 1.27)
+				)
+				(hide yes)
+			)
+		)
+		(property "Datasheet" "http://www.intersil.com/content/dam/Intersil/documents/cd40/cd4000bms-01bms-02bms-25bms.pdf"
+			(at 63.5 132.08 0)
+			(effects
+				(font
+					(size 1.27 1.27)
+				)
+				(hide yes)
+			)
+		)
+		(property "Description" "Quad Nor 2 inputs"
+			(at 63.5 132.08 0)
+			(effects
+				(font
+					(size 1.27 1.27)
+				)
+				(hide yes)
+			)
+		)
+		(pin "3"
+		)
+		(pin "6"
+		)
+		(pin "4"
+		)
+		(pin "9"
+		)
+		(pin "1"
+		)
+		(pin "12"
+		)
+		(pin "5"
+		)
+		(pin "13"
+		)
+		(pin "2"
+		)
+		(pin "11"
+		)
+		(pin "10"
+		)
+		(pin "8"
+		)
+		(pin "7"
+		)
+		(pin "14"
+		)
+		(instances
+			(project ""
+				(path "/d602fbc7-2a38-4026-b8f4-783c9aa802a9"
+					(reference "U2")
+					(unit 1)
+				)
+			)
 		)
 	)
